File: PC104-Breakout/PC104-Breakout.kicad_sch (KiCad schematic)
At the start: 52 parts, among them J1 H1-02x26_Even, J2 H1-02x26_Odd, J3 H2-0x26_Even, J4 Screw_Terminal_01x02, J5 Screw_Terminal_01x02, J6 Screw_Terminal_01x02, J7 Conn_01x02, J8 Conn_01x02, J9 Conn_01x02, M1 MountingHole_Pad, M10 MountingHole_Pad, M11 MountingHole_Pad, M12 MountingHole_Pad, M2 MountingHole_Pad, M3 MountingHole_Pad, M4 MountingHole_Pad, M5 MountingHole_Pad, M6 MountingHole_Pad, M7 MountingHole_Pad, M8 MountingHole_Pad, M9 MountingHole_Pad

Commit message: Polish 3d models, silkscreen
Parts:
- added D7, D8: LED, LED_SMD:LED_0603_1608Metric_Pad1.05x0.95mm_HandSolder, symbol Device:LED
- added J11, J12, J13: Conn_01x03_Socket, Connector_PinSocket_2.54mm:PinSocket_1x03_P2.54mm_Vertical, symbol Connector:Conn_01x03_Socket
- added R15: 5k1, Resistor_SMD:R_0603_1608Metric_Pad0.98x0.95mm_HandSolder, symbol Device:R
- added R16: 3k3, Resistor_SMD:R_0603_1608Metric_Pad0.98x0.95mm_HandSolder, symbol Device:R
- H1: renamed from H2; footprint Connector_PinHeader_2.54mm:PinHeader_2x26_P2.54mm_Vertical -> PC104-Breakout-Lib:PinSocket_2x26_P2.54mm_Vertical_TightPlacement
- H2: renamed from H1; footprint Connector_PinHeader_2.54mm:PinHeader_2x26_P2.54mm_Vertical -> PC104-Breakout-Lib:PinSocket_2x26_P2.54mm_Vertical_TightPlacement
- J1, J2, J3: footprint Connector_PinHeader_2.54mm:PinHeader_2x26_P2.54mm_Vertical -> PC104-Breakout-Lib:PinHeader_2x26_P2.54mm_Vertical_HeaderAndSocket
- J10: renamed from J9; symbol Connector_Generic:Conn_01x03 -> Connector:Conn_01x03_Pin
- J4: renamed from H3; footprint Connector_PinHeader_2.54mm:PinHeader_2x26_P2.54mm_Vertical -> PC104-Breakout-Lib:PinHeader_2x26_P2.54mm_Vertical_HeaderAndSocket
- J8: renamed from J7; symbol Connector_Generic:Conn_01x03 -> Connector:Conn_01x03_Pin
- J9: renamed from J8; symbol Connector_Generic:Conn_01x03 -> Connector:Conn_01x03_Pin
- renumbered D1 to D-H2-25, D2 to D-H2-26, D3 to D-H2-27, D4 to D-H2-28, D5 to D-H2-45, D6 to D-H2-46, J4 to J5, J5 to J6, J6 to J7, R11 to R10, R13 to R11, R10 to R12, R12 to R13
Connections:
- net +3V3: now also J13.1 (Pin_1), J13.2 (Pin_2), J13.3 (Pin_3), R16.1
- net +5V: now also J12.1 (Pin_1), J12.2 (Pin_2), J12.3 (Pin_3), R15.1
- net GND: now also D7.1 (K), D8.1 (K), J11.1 (Pin_1), J11.2 (Pin_2), J11.3 (Pin_3)
- new net: D7.2 (A), R15.2
- new net: D8.2 (A), R16.2
Other:
- note added: "(for breakout pins)"
- moved on the sheet: J5, J6, J7, TP4, TP5, TP6
